File: 03 circuit design/Micromouse_current_all_parts.kicad_pcb (KiCad board)
At the start: 2 copper layers, 80 x 56 mm, 26 parts, among them J1 BATT_IN, J10 RIGHT, J2 UBEC_UNREG, J3 UBEC_REG, J4 R_MOTOR, J5 L_MOTOR, J6 I2C_0, J7 I2C_1, J8 LEFT, J9 FORWARD, Q1 SL2301S, SW1 GF_123-0054, U1 TB6612_DUAL_MOTOR_DRIVER

Commit message: Final Schematic Update
Contains the pcb design files sent for fabrication
Parts:
- added C1: 100nF, Capacitor_SMD:C_1206_3216Metric, F.Cu at (149.0, 115.0)
- added C7: 100nf, Capacitor_SMD:C_0603_1608Metric, F.Cu at (178.5, 95.0)
- added R7: 10K, Resistor_SMD:R_1206_3216Metric, F.Cu at (177.5, 91.0)
- added SW2: SW_SPST, Button_Switch_SMD:SW_SPST_PTS810, F.Cu at (182.0, 92.5)
- moved J6 45.5 mm to (138.8, 122.0)
- moved J7 45.5 mm to (138.0, 76.5)
- moved R2 3.83 mm to (176.3, 98.5)
- moved R3 3.83 mm to (179.5, 98.5)
- moved R4 3.83 mm to (182.8, 98.5)
- moved D3 3.32 mm to (179.0, 105.5)
- moved D4 3.32 mm to (179.0, 112.1)
- moved D5 3.32 mm to (179.0, 118.6)
- moved D2 3.04 mm to (138.0, 115.5)
- moved J3 3.04 mm to (138.5, 108.0)
- moved Q1 3.04 mm to (145.0, 115.5)
- moved R1 3.04 mm to (145.0, 111.5)
- moved J9 1.74 mm to (179.0, 84.0)
Connections:
- A1 pad 12: unconnected-(A1-GPIO9-Pad12) -> /BUTTON
- J6 pad 3: /I2C1_SDA -> /I2C0_SDA
- J6 pad 4: /I2C1_SCL -> /I2C0_SCL
- J6 pad MP: (no net) -> unconnected-(J6-Mount_Pad-PadMP)
- J7 pad 3: /I2C0_SDA -> /I2C1_SDA
- J7 pad 4: /I2C0_SCL -> /I2C1_SCL
- J7 pad MP: (no net) -> unconnected-(J7-Mount_Pad-PadMP)_1
Routing:
- net +3V3: track 94.6 -> 129.5 mm, vias 1 -> 2
- net /BUTTON: track 0.00 -> 21.2 mm
- net GND: track 56.6 -> 73.3 mm, vias 3 -> 0
- net /LED_RED: track 12.7 -> 9.32 mm
- net VSYS: track 7.46 -> 10.9 mm
- net VBUS: track 20.9 -> 24.0 mm
- net /LED_GREEN: track 6.88 -> 7.98 mm
- net /LED_YELLOW: track 8.52 -> 7.66 mm
- net /SHUT_FORWARD: track 7.11 -> 7.78 mm
- net Net-(D5-K): track 20.7 -> 20.2 mm
- net Net-(D4-K): track 14.1 -> 13.5 mm
- net Net-(D3-K): track 7.19 -> 6.67 mm
